Commit message: Scale robot model to 230mm square footprint

File: src/cargo_robot_description/urdf/cargo_robot_1.urdf (robot description, URDF)
Before this commit: robot cargo_robot_1, 5 links, 4 joints
Links:
- link base_link: geometry collision box size=0.18 0.19 0.11; visual box size=0.18 0.19 0.11
- link front_left_wheel: geometry collision sphere radius=0.05; visual cylinder length=0.04 radius=0.05
- link front_right_wheel: geometry collision sphere radius=0.05; visual cylinder length=0.04 radius=0.05
- link rear_left_wheel: geometry collision sphere radius=0.05; visual cylinder length=0.04 radius=0.05
- link rear_right_wheel: geometry collision sphere radius=0.05; visual cylinder length=0.04 radius=0.05
Joints:
- joint front_left_wheel_joint: origin xyz=0.3 0.325 0.1 rpy=-1.5708 0 0 -> xyz=0.065 0.095 0.05 rpy=-1.5708 0 0
- joint front_right_wheel_joint: origin xyz=0.3 -0.325 0.1 rpy=-1.5708 0 0 -> xyz=0.065 -0.095 0.05 rpy=-1.5708 0 0
- joint rear_left_wheel_joint: origin xyz=-0.3 0.325 0.1 rpy=-1.5708 0 0 -> xyz=-0.065 0.095 0.05 rpy=-1.5708 0 0
- joint rear_right_wheel_joint: origin xyz=-0.3 -0.325 0.1 rpy=-1.5708 0 0 -> xyz=-0.065 -0.095 0.05 rpy=-1.5708 0 0

File: src/cargo_robot_description/urdf/cargo_robot_2.urdf (robot description, URDF)
Before this commit: robot cargo_robot_2, 5 links, 4 joints
Links:
- link base_link: geometry collision box size=0.18 0.19 0.11; visual box size=0.18 0.19 0.11
- link front_left_wheel: geometry collision sphere radius=0.05; visual cylinder length=0.04 radius=0.05
- link front_right_wheel: geometry collision sphere radius=0.05; visual cylinder length=0.04 radius=0.05
- link rear_left_wheel: geometry collision sphere radius=0.05; visual cylinder length=0.04 radius=0.05
- link rear_right_wheel: geometry collision sphere radius=0.1; visual sphere radius=0.05
Joints:
- joint front_left_wheel_joint: origin xyz=0.3 0.325 0.1 rpy=-1.5708 0 0 -> xyz=0.065 0.095 0.05 rpy=-1.5708 0 0
- joint front_right_wheel_joint: origin xyz=0.3 -0.325 0.1 rpy=-1.5708 0 0 -> xyz=0.065 -0.095 0.05 rpy=-1.5708 0 0
- joint rear_left_wheel_joint: origin xyz=-0.3 0.325 0.1 rpy=-1.5708 0 0 -> xyz=-0.065 0.095 0.05 rpy=-1.5708 0 0
- joint rear_right_wheel_joint: origin xyz=-0.3 -0.325 0.1 rpy=-1.5708 0 0 -> xyz=-0.065 -0.095 0.05 rpy=-1.5708 0 0

Commit message: Model 60mm wheels and full robot footprint

File: src/cargo_robot_description/urdf/cargo_robot_1.urdf (robot description, URDF)
Before this commit: robot cargo_robot_1, 5 links, 4 joints
Links:
- link base_link: geometry collision box size=0.23 0.23 0.10; visual box size=0.23 0.23 0.10
- link front_left_wheel: geometry collision sphere radius=0.03; visual cylinder length=0.06 radius=0.03
- link front_right_wheel: geometry collision sphere radius=0.03; visual cylinder length=0.06 radius=0.03
- link rear_left_wheel: geometry collision sphere radius=0.03; visual cylinder length=0.06 radius=0.03
- link rear_right_wheel: geometry collision sphere radius=0.03; visual cylinder length=0.06 radius=0.03
Joints:
- joint front_left_wheel_joint: origin xyz=0.065 0.095 0.05 rpy=-1.5708 0 0 -> xyz=0.145 0.145 0.03 rpy=-1.5708 0 0
- joint front_right_wheel_joint: origin xyz=0.065 -0.095 0.05 rpy=-1.5708 0 0 -> xyz=0.145 -0.145 0.03 rpy=-1.5708 0 0
- joint rear_left_wheel_joint: origin xyz=-0.065 0.095 0.05 rpy=-1.5708 0 0 -> xyz=-0.145 0.145 0.03 rpy=-1.5708 0 0
- joint rear_right_wheel_joint: origin xyz=-0.065 -0.095 0.05 rpy=-1.5708 0 0 -> xyz=-0.145 -0.145 0.03 rpy=-1.5708 0 0

File: src/cargo_robot_description/urdf/cargo_robot_2.urdf (robot description, URDF)
Before this commit: robot cargo_robot_2, 5 links, 4 joints
Links:
- link base_link: geometry collision box size=0.23 0.23 0.10; visual box size=0.23 0.23 0.10
- link front_left_wheel: geometry collision sphere radius=0.03; visual cylinder length=0.06 radius=0.03
- link front_right_wheel: geometry collision sphere radius=0.03; visual cylinder length=0.06 radius=0.03
- link rear_left_wheel: geometry collision sphere radius=0.03; visual cylinder length=0.06 radius=0.03
- link rear_right_wheel: geometry collision sphere radius=0.03; visual cylinder length=0.06 radius=0.03
Joints:
- joint front_left_wheel_joint: origin xyz=0.065 0.095 0.05 rpy=-1.5708 0 0 -> xyz=0.145 0.145 0.03 rpy=-1.5708 0 0
- joint front_right_wheel_joint: origin xyz=0.065 -0.095 0.05 rpy=-1.5708 0 0 -> xyz=0.145 -0.145 0.03 rpy=-1.5708 0 0
- joint rear_left_wheel_joint: origin xyz=-0.065 0.095 0.05 rpy=-1.5708 0 0 -> xyz=-0.145 0.145 0.03 rpy=-1.5708 0 0
- joint rear_right_wheel_joint: origin xyz=-0.065 -0.095 0.05 rpy=-1.5708 0 0 -> xyz=-0.145 -0.145 0.03 rpy=-1.5708 0 0

Commit message: Place mecanum wheels along robot sides

File: src/cargo_robot_description/urdf/cargo_robot_1.urdf (robot description, URDF)
Before this commit: robot cargo_robot_1, 5 links, 4 joints
Joints:
- joint front_left_wheel_joint: origin xyz=0.145 0.145 0.03 rpy=-1.5708 0 0 -> xyz=0.075 0.145 0.03 rpy=-1.5708 0 0
- joint front_right_wheel_joint: origin xyz=0.145 -0.145 0.03 rpy=-1.5708 0 0 -> xyz=0.075 -0.145 0.03 rpy=-1.5708 0 0
- joint rear_left_wheel_joint: origin xyz=-0.145 0.145 0.03 rpy=-1.5708 0 0 -> xyz=-0.075 0.145 0.03 rpy=-1.5708 0 0
- joint rear_right_wheel_joint: origin xyz=-0.145 -0.145 0.03 rpy=-1.5708 0 0 -> xyz=-0.075 -0.145 0.03 rpy=-1.5708 0 0

File: src/cargo_robot_description/urdf/cargo_robot_2.urdf (robot description, URDF)
Before this commit: robot cargo_robot_2, 5 links, 4 joints
Joints:
- joint front_left_wheel_joint: origin xyz=0.145 0.145 0.03 rpy=-1.5708 0 0 -> xyz=0.075 0.145 0.03 rpy=-1.5708 0 0
- joint front_right_wheel_joint: origin xyz=0.145 -0.145 0.03 rpy=-1.5708 0 0 -> xyz=0.075 -0.145 0.03 rpy=-1.5708 0 0
- joint rear_left_wheel_joint: origin xyz=-0.145 0.145 0.03 rpy=-1.5708 0 0 -> xyz=-0.075 0.145 0.03 rpy=-1.5708 0 0
- joint rear_right_wheel_joint: origin xyz=-0.145 -0.145 0.03 rpy=-1.5708 0 0 -> xyz=-0.075 -0.145 0.03 rpy=-1.5708 0 0

Commit message: Stabilize mecanum wheel ground contact

File: src/cargo_robot_description/urdf/cargo_robot_1.urdf (robot description, URDF)
Before this commit: robot cargo_robot_1, 5 links, 4 joints
Links:
- link front_left_wheel: geometry collision cylinder length=0.06 radius=0.03; visual cylinder length=0.06 radius=0.03
- link front_right_wheel: geometry collision cylinder length=0.06 radius=0.03; visual cylinder length=0.06 radius=0.03
- link rear_left_wheel: geometry collision cylinder length=0.06 radius=0.03; visual cylinder length=0.06 radius=0.03
- link rear_right_wheel: geometry collision cylinder length=0.06 radius=0.03; visual cylinder length=0.06 radius=0.03

File: src/cargo_robot_description/urdf/cargo_robot_2.urdf (robot description, URDF)
Before this commit: robot cargo_robot_2, 5 links, 4 joints
Links:
- link front_left_wheel: geometry collision cylinder length=0.06 radius=0.03; visual cylinder length=0.06 radius=0.03
- link front_right_wheel: geometry collision cylinder length=0.06 radius=0.03; visual cylinder length=0.06 radius=0.03
- link rear_left_wheel: geometry collision cylinder length=0.06 radius=0.03; visual cylinder length=0.06 radius=0.03
- link rear_right_wheel: geometry collision cylinder length=0.06 radius=0.03; visual cylinder length=0.06 radius=0.03
